Commit message: Update to xacro:property

File: husky_description/urdf/husky.urdf.xacro (robot description, xacro)
@@ -33,9 +33,9 @@
   <xacro:include filename="$(find flir_ptu_description)/urdf/d46.urdf.xacro"/>
   <xacro:include filename="$(find pointgrey_camera_description)/urdf/pointgrey_bumblebee2.urdf.xacro"/>
-  <property name="M_PI" value="3.14159"/>
+  <xacro:property name="M_PI" value="3.14159"/>
   <!-- Base Size -->
-  <property name="base_x_size" value="0.98740000" />
-  <property name="base_y_size" value="0.57090000" />
-  <property name="base_z_size" value="0.24750000" />
+  <xacro:property name="base_x_size" value="0.98740000" />
+  <xacro:property name="base_y_size" value="0.57090000" />
+  <xacro:property name="base_z_size" value="0.24750000" />
   <!-- Wheel Mounting Positions -->
   <xacro:property name="wheelbase" value="0.5120" />

Commit message: Remove point_grey cam

File: husky_description/urdf/husky.urdf.xacro (robot description, xacro)
@@ -32,5 +32,5 @@
   <xacro:include filename="$(find robotiq_force_torque_sensor)/urdf/robotiq_fts300.urdf.xacro"/>
   <xacro:include filename="$(find flir_ptu_description)/urdf/d46.urdf.xacro"/>
-  <xacro:include filename="$(find pointgrey_camera_description)/urdf/pointgrey_bumblebee2.urdf.xacro"/>
+  <!--xacro:include filename="$(find pointgrey_camera_description)/urdf/pointgrey_bumblebee2.urdf.xacro"/>-->
   <xacro:property name="M_PI" value="3.14159"/>
   <!-- Base Size -->
@@ -132,10 +132,10 @@
         </joint>
         <!-- Add bumblebee camera -->
-       <BB2-08S2C-38 frame="bumblebee2" name="bumblebee2" />
+       <!-- <BB2-08S2C-38 frame="bumblebee2" name="bumblebee2" />
         <joint name="bumblebee2_mount_joint" type="fixed">
            <origin xyz="0 0 0.00" rpy="0 0 0" />
            <parent link="husky_ptu_mount_link" />
            <child link="bumblebee2" />
-        </joint>
+        </joint> -->
        <xacro:if value="$(optenv ROBOTIQ_GRIPPERS_WITH_FT_ENABLED false)">
             <!-- Add force torque model FT300 -->

Commit message: Commented out the gripper portion from the urdf

File: husky_description/urdf/husky.urdf.xacro (robot description, xacro)
@@ -176,5 +176,5 @@
   </xacro:macro>
    <!-- Collision prevention boxes to prevent hitting the cables -->
-  <link name="l_gripper_protection_box">
+  <!-- <link name="l_gripper_protection_box">
     <visual>
       <origin xyz="0.04 0 0" rpy="0 0 0" />
@@ -189,7 +189,7 @@
       </geometry>
     </collision>
-  </link>
+  </link> -->
   <!-- Collision prevention boxes to prevent hitting the cables -->
-  <link name="r_gripper_protection_box">
+  <!-- <link name="r_gripper_protection_box">
     <visual>
       <origin xyz="0.04 0 0" rpy="0 0 0" />
@@ -209,10 +209,10 @@
     <child link="l_gripper_protection_box" />
     <origin xyz="0 0 0" rpy="0 0 0" />
-  </joint>
+  </joint> -->
   <!-- Attach the boxes to the gripper to prevent collisions -->
-  <joint name="r_gripper_protection" type="fixed">
+  <!-- <joint name="r_gripper_protection" type="fixed">
     <parent link="r_palm" />
     <child link="r_gripper_protection_box" />
     <origin xyz="0 0 0" rpy="0 0 0" />
-  </joint>
+  </joint> -->
 </robot>
